Commit message: .

File: Ros_Drive/amr_urdf/urdf/robot.urdf (robot description, URDF)
Before this commit: robot AMR, 16 links, 15 joints
Links:
- link base_link: geometry collision mesh filename=package://amr_urdf/meshes/body.stl scale=0.001 0.001 0.001; visual mesh filename=package://amr_urdf/meshes/body.stl scale=0.001 0.001 0.001
- link camera_link: geometry collision mesh filename=package://amr_urdf/meshes/depth_camera.stl scale=0.001 0.001 0.001; visual mesh filename=package://amr_urdf/meshes/depth_camera.stl scale=0.001 0.001 0.001
- link gripper_base: geometry collision mesh filename=package://amr_urdf/meshes/gripper_base.stl scale=1 1 1; visual mesh filename=package://amr_urdf/meshes/gripper_base.stl scale=1 1 1
- link gripper_fix: geometry collision mesh filename=package://amr_urdf/meshes/gripper_fix.stl scale=1 1 1; visual mesh filename=package://amr_urdf/meshes/gripper_fix.stl scale=1 1 1
- link gripper_movable: geometry collision mesh filename=package://amr_urdf/meshes/gripper_movable.stl scale=1 1 1; visual mesh filename=package://amr_urdf/meshes/gripper_movable.stl scale=1 1 1
- link laser_link: geometry collision mesh filename=package://amr_urdf/meshes/rplidar-a2.stl scale=1 1 1; visual mesh filename=package://amr_urdf/meshes/rplidar-a2.stl scale=1 1 1
- link left_wheel: geometry collision mesh filename=package://amr_urdf/meshes/wheel.stl scale=0.001 0.001 0.001; visual mesh filename=package://amr_urdf/meshes/wheel.stl scale=0.001 0.001 0.001
- link link1: geometry collision mesh filename=package://amr_urdf/meshes/base.stl scale=1 1 1; visual mesh filename=package://amr_urdf/meshes/base.stl scale=1 1 1
- link link2: geometry collision mesh filename=package://amr_urdf/meshes/shoulder.stl scale=1 1 1; visual mesh filename=package://amr_urdf/meshes/shoulder.stl scale=1 1 1
- link link3: geometry collision mesh filename=package://amr_urdf/meshes/elbow.stl scale=1 1 1; visual mesh filename=package://amr_urdf/meshes/elbow.stl scale=1 1 1
- link link4: geometry collision mesh filename=package://amr_urdf/meshes/wrist_pitch.stl scale=1 1 1; visual mesh filename=package://amr_urdf/meshes/wrist_pitch.stl scale=1 1 1
- link link5: geometry collision mesh filename=package://amr_urdf/meshes/wrist_roll.stl scale=1 1 1; visual mesh filename=package://amr_urdf/meshes/wrist_roll.stl scale=1 1 1
- link right_wheel: geometry collision mesh filename=package://amr_urdf/meshes/wheel.stl scale=0.001 0.001 0.001; visual mesh filename=package://amr_urdf/meshes/wheel.stl scale=0.001 0.001 0.001
Joints:
- joint imu_joint: parent base_footprint -> base_link
- joint laser_joint: origin xyz=0.2305 0 0.08 rpy=0 0 0 -> xyz=0.2335 0 0.08 rpy=0 0 0
